Commit message: Update Kangaroo Model

File: robots/kangaroo_like_2legs/robot.urdf (robot description, URDF)
Before this commit: robot onshape, 131 links, 130 joints
Links:
- removed link center_hip
- removed link closedloop0_A_3D
- removed link closedloop0_B_3D
- removed link closedloop10_A_3D
- removed link closedloop10_B_3D
- removed link closedloop11_A_3D
- removed link closedloop11_B_3D
- removed link closedloop14_A_3D
- removed link closedloop14_B_3D
- removed link closedloop15_A_3D
- removed link closedloop15_B_3D
- removed link closedloop17_A_6D
- removed link closedloop17_B_6D
- removed link closedloop18_A_6D
- removed link closedloop18_B_6D
- removed link closedloop19_A_6D
- removed link closedloop19_B_6D
- removed link closedloop1_A_3D
- removed link closedloop1_B_3D
- removed link closedloop20_A_3D
- removed link closedloop20_B_3D
- removed link closedloop21_A_3D
- removed link closedloop21_B_3D
- removed link closedloop22_A_3D
- removed link closedloop22_B_3D
- removed link closedloop23_A_3D
- removed link closedloop23_B_3D
- removed link closedloop2_A_3D
- removed link closedloop2_B_3D
- removed link closedloop3_A_6D
- removed link closedloop3_B_6D
- removed link closedloop4_A_6D
- removed link closedloop4_B_6D
- removed link closedloop5_A_6D
- removed link closedloop5_B_6D
- removed link closedloop9_A_3D
- removed link closedloop9_B_3D
- removed link cylinder_10
- removed link cylinder_11
- removed link cylinder_12
- removed link cylinder_13
- removed link cylinder_14
- removed link cylinder_15
- removed link cylinder_16
- removed link cylinder_17
- removed link cylinder_18
- removed link cylinder_19
- removed link cylinder_20
- removed link cylinder_21
- removed link cylinder_22
- removed link cylinder_23
- removed link cylinder_24
- removed link cylinder_5
- removed link cylinder_6
- removed link cylinder_7
- removed link cylinder_8
- removed link cylinder_9
- removed link part_4
- removed link part_4_2
- removed link part_7
- removed link part_7_2
- removed link part_7_3
- removed link part_7_4
- removed link part_7_5
- removed link part_7_6
- removed link part_7_7
- removed link part_7_8
- removed link part_8
- removed link part_8_2
- removed link part_9
- removed link part_9_2
- removed link transmission_ankle
- removed link transmission_ankle2
- removed link transmission_ankle2_2
- removed link transmission_ankle_2
- added link part_4_4rod, mass 0.011311035579799528367; collision mesh filename=package:///part_4_4rod.stl; visual mesh filename=package:///part_4_4rod.stl
- added link part_4_4rod_2, mass 0.011311035579799528367; collision mesh filename=package:///part_4_4rod.stl; visual mesh filename=package:///part_4_4rod.stl
- link hanche_gauche: mass 0.14908820308432116364 -> 0.14908830550245633084
- link hip_part: mass 0.1490882064698049736 -> 0.14908831103070877
- link part_1: mass 0.24432174426363428843 -> 0.24432174426363423292
- link part_3: mass 0.20213480893965668495 -> 0.2021348089396567127
- link part_3_2: mass 0.20213480893965668495 -> 0.2021348089396567127
Joints:
- removed joint center_hip_frame
- removed joint closedloop0_A_3D_frame
- removed joint closedloop0_B_3D_frame
- removed joint closedloop10_A_3D_frame
- removed joint closedloop10_B_3D_frame
- removed joint closedloop11_A_3D_frame
- removed joint closedloop11_B_3D_frame
- removed joint closedloop14_A_3D_frame
- removed joint closedloop14_B_3D_frame
- removed joint closedloop15_A_3D_frame
- removed joint closedloop15_B_3D_frame
- removed joint closedloop17_A_6D_frame
- removed joint closedloop17_B_6D_frame
- removed joint closedloop18_A_6D_frame
- removed joint closedloop18_B_6D_frame
- removed joint closedloop19_A_6D_frame
- removed joint closedloop19_B_6D_frame
- removed joint closedloop1_A_3D_frame
- removed joint closedloop1_B_3D_frame
- removed joint closedloop20_A_3D_frame
- removed joint closedloop20_B_3D_frame
- removed joint closedloop21_A_3D_frame
- removed joint closedloop21_B_3D_frame
- removed joint closedloop22_A_3D_frame
- removed joint closedloop22_B_3D_frame
- removed joint closedloop23_A_3D_frame
- removed joint closedloop23_B_3D_frame
- removed joint closedloop2_A_3D_frame
- removed joint closedloop2_B_3D_frame
- removed joint closedloop3_A_6D_frame
- removed joint closedloop3_B_6D_frame
- removed joint closedloop4_A_6D_frame
- removed joint closedloop4_B_6D_frame
- removed joint closedloop5_A_6D_frame
- removed joint closedloop5_B_6D_frame
- removed joint closedloop9_A_3D_frame
- removed joint closedloop9_B_3D_frame
- removed joint free_spherical_hip_xy_1_left
- removed joint free_spherical_hipxy_2_left
- removed joint free_spherical_motor_holder_hipz
- removed joint motor_ankle1
- removed joint motor_ankle1_left
- removed joint motor_ankle2
- removed joint motor_ankle2_left
- removed joint motor_hip_xy_1
- removed joint motor_hip_xy_1_left
- removed joint motor_hip_xy_2
- removed joint motor_hip_xy_2_left
- removed joint motor_hip_z_left
- removed joint motor_hipz
- removed joint spherical_free_hip_left
- removed joint spherical_lower_hip1
- removed joint spherical_lower_hip2
- removed joint spherical_motor_transmission_hip1_left
- removed joint spherical_motor_transmission_hip2_left
- removed joint spherical_transmission_foot1
- removed joint spherical_transmission_foot1_left
- removed joint spherical_transmission_foot2
- removed joint spherical_transmission_foot2_left
- removed joint spherical_transmission_hip3
- removed joint spherical_transmission_hip3_left
- removed joint spherical_transmission_hip4
- removed joint spherical_transmission_hip4_left
- removed joint spherical_transmission_motor_hip1
- removed joint spherical_transmission_motor_hip2
- removed joint transmission_1_knee_left
- removed joint transmission_2_knee_left
- removed joint transmission_ankle3_left
- removed joint transmission_ankle4_left
- removed joint transmission_hip1
- removed joint transmission_hip2
- removed joint triangle_knee1
- removed joint triangle_knee2
- joint 4rod_knee: child part_4_2 -> part_4_4rod_2; origin xyz=0.046047631733746152705 -0.019483726843523285766 -1.1102230246251565404e-16 rpy=3.141592653589793116 2.0222300709232764069e-16 -1.2672660179280783588 -> xyz=0.046047631733745819638 -0.019483726843523424543 2.7755575615628913511e-16 rpy=3.141592653589793116 2.106906146808720801e-16 -1.2660224049965986826
- joint 4rof_knee_left: child part_4 -> part_4_4rod; origin xyz=0.046047631733745944538 -0.019483726843523313521 1.9428902930940239457e-16 rpy=-3.141592653589793116 -3.6494643439707380228e-16 -1.3191803600776987881 -> xyz=0.046047631733746013927 -0.019483726843523313521 -1.0408340855860842566e-17 rpy=3.1415926535897926719 1.1366954211112319194e-16 -1.2672660179279957582
- joint closedloop12_A_3D_frame: origin xyz=0 -6.9388939039072283776e-18 -0.42720000000000002416 rpy=-3.141592653589793116 1.5073519112078350571e-17 -7.4426580352851623595e-17 -> xyz=-1.1102230246251565404e-16 0 -0.42720000000000002416 rpy=-3.1415926535897926719 -2.7014521880793210558e-16 -4.051566801923114862e-16
- joint closedloop12_B_3D_frame: origin xyz=0.038967453687049735667 -0.092095263467496732424 -6.2450045135165055399e-17 rpy=-1.57079632679489678 -2.1358826958981862826e-17 3.141592653589793116 -> xyz=0.038967453687049818933 -0.092095263467496676912 -3.4694469519536141888e-18 rpy=-1.57079632679489678 2.7152200089216079401e-27 3.1415926535897926719; parent part_4 -> part_4_4rod
- joint closedloop13_A_3D_frame: origin xyz=-2.7755575615628913511e-17 -3.4694469519536141888e-18 -0.1414199999999999624 rpy=3.141592653589793116 4.7221641683567358421e-17 -4.15595262285446502e-18 -> xyz=0 0 -0.14141999999999999016 rpy=-3.141592653589793116 -3.025217164274315018e-16 -7.074917909937649877e-18
- joint closedloop13_B_3D_frame: origin xyz=0.083867056794542468867 0.0077119035015027481705 -0.071500000000000007994 rpy=1.570796326794896558 4.3024590727307537194e-19 3.141592653589793116 -> xyz=0.083867056794542468867 0.007711903501502720415 -0.071500000000000035749 rpy=1.570796326794896558 1.4106605912204471211e-29 3.141592653589793116
- joint closedloop16_A_3D_frame: origin xyz=-1.6653345369377348106e-16 4.6837533851373791549e-17 -0.021999999999999755862 rpy=4.3690578280789386181e-19 9.2082750998859503317e-18 -2.9498235737414757909e-16 -> xyz=0 -1.3877787807814456755e-17 -0.02200000000000001954 rpy=5.3987244821969968243e-16 -8.2507344659508689231e-16 -1.1134981280911585485e-15; parent cylinder_6 -> cylinder_2
- joint closedloop16_B_3D_frame: origin xyz=6.9388939039072283776e-18 -2.7755575615628913511e-17 -0.022000000000000033418 rpy=3.141592653589793116 -6.6420938655515744184e-17 -1.570796326794896558 -> xyz=-3.4694469519536141888e-18 0 -0.022000000000000075051 rpy=3.141592653589793116 1.5645422202668635312e-16 -1.570796326794896558; parent cylinder_3 -> cylinder
- joint closedloop6_A_3D_frame: origin xyz=0.038967453687049735667 -0.092095263467496635279 0 rpy=1.570796326794896558 4.0264892395916754221e-23 -1.570796326794896336 -> xyz=0.038967453687049874445 -0.092095263467496676912 -1.1102230246251565404e-16 rpy=1.570796326794896558 -8.1969636802554788053e-29 -1.570796326794896336; parent part_4_2 -> part_4_4rod_2
- joint closedloop6_B_3D_frame: origin xyz=0 5.5511151231257827021e-17 -0.42719999999999985762 rpy=-3.1415926535897926719 4.4452919195117772876e-16 -3.141592653589793116 -> xyz=3.8857805861880478915e-16 -1.1102230246251565404e-16 -0.42719999999999996865 rpy=3.141592653589793116 -6.9431862954624840017e-17 -1.57079632679489678
- joint closedloop7_A_3D_frame: origin xyz=-5.5511151231257827021e-17 5.5511151231257827021e-17 -0.14142000000000004567 rpy=-3.141592653589793116 -3.3269411146025779664e-16 1.6049846913326267147e-16 -> xyz=-2.7755575615628913511e-17 0 -0.14142000000000004567 rpy=-3.1415926535897926719 -6.6400050883493334936e-16 -2.3979609692655224185e-16
- joint closedloop7_B_3D_frame: origin xyz=0.083867056794542399478 -0.0077119035015026926594 -0.071500000000000063505 rpy=1.570796326794896558 -1.1282895733432249803e-30 -1.3863489958700578838e-14 -> xyz=0.083867056794542371723 -0.007711903501502720415 -0.071500000000000063505 rpy=1.570796326794896558 -1.5978176936970281056e-30 -1.3878092409244805529e-14
- joint closedloop8_A_3D_frame: origin xyz=2.7755575615628913511e-16 1.1102230246251565404e-16 -0.022000000000000227707 rpy=-3.141592653589793116 4.2576220938315339428e-17 -1.570796326794896336 -> xyz=0 0 -0.022000000000000033418 rpy=3.141592653589793116 -1.7853591269876519938e-16 -1.570796326794896558; parent cylinder_14 -> cylinder_3
- joint closedloop8_B_3D_frame: origin xyz=5.5511151231257827021e-17 5.5511151231257827021e-17 -0.02200000000000001954 rpy=1.0380387903692397796e-15 -3.3350635930275230669e-16 1.5707963267948978903 -> xyz=-1.3877787807814456755e-17 0 -0.022000000000000061173 rpy=6.0378406373761762468e-15 -4.3612875086825312607e-16 1.570796326794896558; parent cylinder_17 -> cylinder_4
- joint foot_left_frame: origin xyz=0.012016949221079833987 0.038500000000000089706 6.8117394433353517513e-09 rpy=1.570796326794896558 -1.2589951705659949766e-17 -1.4953607374009730393e-14 -> xyz=0.012016949221079764598 0.038499999999999867661 6.8117394502742456552e-09 rpy=1.570796326794896558 -1.990244812700938893e-32 1.6446679738098929258e-17
- joint foot_right_frame: origin xyz=0.012016949221079833987 0.038499999999999978684 6.811739394763094424e-09 rpy=1.5707963267948974462 8.530342469776898909e-19 1.4132086598801471662e-15 -> xyz=0.012016949221079709087 0.038500000000000200728 6.8117392282296407302e-09 rpy=1.5707963267948978903 2.0539125955564721522e-15 -6.9014379821604008548e-16
- joint frame_motor_ankle1: origin xyz=0.054086706326755190632 0.014047405294960846334 -0.11824999999999996625 rpy=-1.57079632679489678 0.17393610028771827603 0.2858933777993311609 -> xyz=0.054086706326755197571 0.014047405294960818578 -0.11825000000000002176 rpy=1.570796326794896558 3.4767615064910652246e-30 -2.8556992757904686719; type revolute -> fixed
- joint frame_motor_ankle1_left: origin xyz=0.05408670632675532941 -0.014047405294960790823 -0.11825000000000007727 rpy=1.570796326794896336 -0.0082317284983713604612 -0.28589337779933193806 -> xyz=0.054086706326755336349 -0.014047405294960790823 -0.11825000000000000788 rpy=1.570796326794896558 5.1626054294143844551e-27 -0.28589337779932444406; type revolute -> fixed
- joint frame_motor_ankle2: origin xyz=0.054086706326755183694 0.014047405294960790823 -0.024750000000000021982 rpy=1.57079632679489678 -0.077730067950898998341 -2.8556992757904731128 -> xyz=0.054086706326755100427 0.014047405294960790823 -0.024749999999999994227 rpy=-1.2849029489955836603 -1.5707963267948792385 0; type revolute -> fixed
- joint frame_motor_ankle2_left: origin xyz=0.054086706326755273899 -0.014047405294960818578 -0.02474999999999997341 rpy=-1.5707963267948972241 -0.11316607510714726814 2.8556992757904873237 -> xyz=0.054086706326755301655 -0.014047405294960735311 -0.024750000000000021982 rpy=-1.570796326794896558 -1.7314630718498674831e-30 2.8556992757904686719; type revolute -> fixed
- joint frame_motor_knee: origin xyz=-0.061655078133537100094 -0.018724201373191834419 4.2972847502653621632e-12 rpy=1.5707963267948970021 1.1013926676990786202 2.5355753428775891223 -> xyz=-0.061655078133537349894 -0.018724201373191723397 4.297340261416593421e-12 rpy=1.570796326794896558 -4.5884075768098473358e-30 2.5355753428775971159; type revolute -> fixed
- joint free_ankle_universal_x_left: origin xyz=6.6000000000010494716e-05 1.1102230246251565404e-16 6.5999999999982739141e-05 rpy=1.570796326794896558 -1.2724678177825976544 1.5707963267948641395 -> xyz=6.6000000000000086375e-05 0 6.5999999999982739141e-05 rpy=-1.5707963267949025532 -1.3119332803331693604 -1.5707963267948907848
- joint free_ankle_universalx: origin xyz=6.6000000000066005867e-05 1.1102230246251565404e-16 6.5999999999954983565e-05 rpy=1.570796326794896558 -1.2632158641075659222 1.5707963267949021091 -> xyz=6.6000000001009695438e-05 2.2204460492503130808e-16 6.599999999973293896e-05 rpy=-1.5707963267948881203 -1.3214621537091344461 -1.5707963267948723551
- joint free_hip_left: origin xyz=0.012500000000000019776 0.044999999999999928946 -0.0049999999999998934186 rpy=3.2497958717751232591e-17 -7.9160110916992996937e-16 -0.013408965559009784763 -> xyz=0.012500000000000018041 0.044999999999999928946 -0.0049999999999998934186 rpy=1.4983823821050141706e-17 -8.5099172879074144489e-16 -2.7755575615627912643e-16
- joint free_motor_holder_1: origin xyz=0.012500000000000002429 -0.037124999999999686029 -0.077000000000000040634 rpy=1.57079632679489678 -0.021206259450683103557 -1.5707963267948974462 -> xyz=0.012500000000000165493 -0.03712500000000068523 -0.076999999999999707567 rpy=1.570796326794896558 -4.834667595244735176e-18 -1.5707963267948970021; type revolute -> fixed
- joint free_motor_holder_1_left: origin xyz=0.012500000000000002429 -0.037124999999999935829 -0.076999999999999957367 rpy=1.570796326794896558 -0.029014515778508449817 -1.5707963267948918951 -> xyz=0.012500000000000005898 -0.037124999999999901135 -0.077000000000000082268 rpy=1.570796326794896558 -2.0029671421627252872e-31 -1.570796326794896558; type revolute -> fixed
- joint free_motor_holder_2: type revolute -> fixed
- joint free_motor_holder_2_left: origin xyz=0.012499999999999960795 0.037125000000000137057 -0.076999999999999971245 rpy=-1.570796326794896558 -0.0048215860931459190303 1.5707963267948970021 -> xyz=0.012500000000000439579 0.037125000000001198708 -0.077000000000000082268 rpy=-1.570796326794896558 -8.8532703001475453083e-19 1.5707963267948958919; type revolute -> fixed
- joint free_motor_holder_3: origin xyz=0.012500000000000037123 0.037125000000000046851 -0.077000000000000484723 rpy=-1.570796326794896558 -0.01926420611835273286 1.5707963267948950037 -> xyz=0.012500000000000151615 0.037125000000000019096 -0.0769999999999983753 rpy=1.570796326794896558 -3.8126966188221397778e-16 -1.5707963267948974462; type revolute -> fixed
- joint free_motor_holder_hip_xy1_left: origin xyz=-2.7755575615628913511e-17 -5.5511151231257827021e-17 -0.055000000000000007216 rpy=-1.5707963267948972241 1.4869452775825180435 1.5707963267949112129 -> xyz=1.3877787807814456755e-17 4.1633363423443370266e-17 -0.055000000000000014155 rpy=3.141592653589793116 1.5707963267948930053 0; type revolute -> fixed
- joint free_motor_holder_hip_xy2_left: origin xyz=3.4694469519536141888e-18 -2.7755575615628913511e-17 -0.055000000000000028033 rpy=-1.570796326794896558 -1.4785663491793541446 1.5707963267948812369 -> xyz=-1.7347234759768070944e-18 -4.1633363423443370266e-17 -0.05500000000000004885 rpy=-0 -1.5707963267948930053 0; type revolute -> fixed
- joint free_motor_holder_hipxy1: origin xyz=5.5511151231257827021e-17 -5.5511151231257827021e-17 -0.055000000000000007216 rpy=-1.5707963267948970021 1.4788923407477159166 1.5707963267949140995 -> xyz=5.5511151231257827021e-17 1.6237011735142914404e-15 -0.055000000000000326406 rpy=-3.7643499428695787037e-16 -1.5707963267948930053 0; type revolute -> fixed
- joint free_motor_holder_hipxy2: origin xyz=0 -6.9388939039072283776e-17 -0.055000000000000007216 rpy=-1.570796326794896558 -1.4788959325010997414 1.5707963267948537034 -> xyz=0 6.9388939039072283776e-17 -0.054999999999999993339 rpy=5.9318642287127407277e-31 -1.570796326794891451 0; type revolute -> fixed
- joint free_motor_knee_left: origin xyz=-0.06165507813353749561 -0.018724201373191556863 4.2973541392044012355e-12 rpy=1.5707963267948976682 1.4446000808328676168 2.5355753428775962277 -> xyz=-0.061655078133537336016 -0.018724201373191695641 4.2973437308635453746e-12 rpy=-0.96477901608270033584 1.570796326794896558 0; type revolute -> fixed
- joint free_spherical_motor_holder_1: origin xyz=-1.3877787807814456755e-17 0 -0.051749999999999886369 rpy=1.570796326794896558 -0.094549574280562209694 1.5707963267948930053 -> xyz=5.5511151231257827021e-17 -5.5511151231257827021e-17 -0.051750000000000330458 rpy=1.570796326794896558 -6.9388939038292651928e-18 1.5707963267948972241; type revolute -> fixed
- joint free_universal_motor_holder_hipz_left: origin xyz=-0.10299999999999671918 0.0064999999999999988343 -1.1102230246251565404e-16 rpy=8.0307403322854623642e-18 8.3515970769616968963e-16 -3.1383830382600423903 -> xyz=-0.1029999999999967053 0.006499999999999950262 -2.2204460492503130808e-16 rpy=5.3604551186845543223e-18 8.3516399299402682153e-16 -3.141592653589793116; type revolute -> fixed
- joint free_universal_x_hip_left: origin xyz=-1.7347234759768070944e-18 6.2450045135165055399e-17 -0.1649999999999999245 rpy=1.570796326794896558 0.059826915957553218617 -1.57079632679489678 -> xyz=-1.7347234759768070944e-17 6.9388939039072283776e-17 -0.16499999999999981348 rpy=1.570796326794896336 -1.1212833847574704648e-16 -1.57079632679489678
- joint free_universal_y_foot_left: origin xyz=0.21747050071614940081 -0.33571800862966411083 1.3877787807814456755e-17 rpy=-1.5707963267948943376 -1.5448377095245018342 1.5707963267950189046 -> xyz=0.2174705007161493453 -0.33571800862966422185 1.3877787807814456755e-17 rpy=-1.5112054271051183109e-15 -1.5707963267948947816 0
- joint free_universal_y_hip_left: origin xyz=-6.5999999999996616928e-05 0 -6.5999999999996616928e-05 rpy=-1.57079632679489678 -1.5206476855511772417 1.5707963267949061059 -> xyz=-6.6000000000010494716e-05 0 -6.5999999999998351652e-05 rpy=-1.570796326794896558 -1.5017238724374586401 1.5707963267948976682
- joint lower_hip: origin xyz=6.6000000000038250292e-05 -2.7755575615628913511e-17 -6.6000000000003555822e-05 rpy=1.5707963267949520692 -1.5388859775008443265 1.5707963267948683583 -> xyz=6.5999999999982739141e-05 -2.7755575615628913511e-17 -6.6000000000277642132e-05 rpy=-1.5707963267957496534 -1.5687216740986209551 -1.5707963267944957675
- joint lower_knee: origin xyz=-0.2174705007161515935 -0.33571800862966272305 0 rpy=2.0331881199897477086e-17 3.2102059775878614431e-15 0.89630439304595999062 -> xyz=-0.21747050071615176003 -0.33571800862966277856 5.5511151231257827021e-17 rpy=2.0331879961906762931e-17 3.4472911644634325801e-17 0.89630439304597675498
- joint lower_knee_left: origin xyz=-0.21747050071615162126 -0.33571800862966283407 0 rpy=-4.1105915432294974674e-16 4.2186246058266865539e-16 0.84062809210853284281 -> xyz=-0.2174705007161515935 -0.33571800862966277856 -1.0408340855860842566e-17 rpy=-1.9453279478922098385e-18 5.6284242543479202598e-17 0.89630439304598807926
- joint motor_knee: child cylinder_14 -> cylinder_3; origin xyz=5.5511151231257827021e-16 2.4286128663675299322e-17 0.0048371488452673555569 rpy=3.141592653589793116 1.2572887915623930455e-15 -4.0658567876216576861e-15 -> xyz=-2.0927704014184200787e-14 0 0.0060390264684015010355 rpy=3.141592653589793116 2.2512629927158492999e-14 1.7262838832682730261e-16
- joint motor_knee_left: child cylinder_3 -> cylinder; origin xyz=-5.1868231931706532123e-16 -1.1102230246251565404e-16 0.0071577726412921510724 rpy=-3.141592653589793116 -2.6517818628931859556e-15 -2.2199395511922745312e-15 -> xyz=-5.4123372450476381346e-16 -1.1102230246251565404e-16 0.0035931979665884822284 rpy=-3.141592653589793116 -1.4811990068826889974e-15 3.1591141143922434355e-16
- joint spherical_4rod: origin xyz=0.019483726843525006611 -0.046047631733748373151 0 rpy=-1.57079632679489678 0.016852862325202326577 -1.5707963267948961139 -> xyz=0.019483726843525034367 -0.046047631733748359273 0 rpy=-1.57079632679489678 0.016852862325203155774 -1.5707963267948981123; parent part_4_2 -> part_4_4rod_2
- joint spherical_4rod_left: origin xyz=0.019483726843524840078 -0.046047631733748359273 -1.3877787807814456755e-17 rpy=1.57079632679489678 0.061687001704508914735 1.5707963267948954478 -> xyz=0.019483726843524978856 -0.046047631733748387028 3.4694469519536141888e-18 rpy=1.57079632679489678 0.02445729775480075599 1.5707963267948901187; parent part_4 -> part_4_4rod
- joint spherical_actuation_knee_left: child cylinder_6 -> cylinder_2; origin xyz=-0.013749999999999797107 -0.0025000000000000022204 -0.070874999999999993561 rpy=1.570796326794896558 -0.15153054045334352073 1.570796326794896336 -> xyz=-0.01374999999999996711 -0.0024999999999999744649 -0.070874999999999993561 rpy=1.570796326794896558 -0.29198081522868968296 1.5707963267948992225
- joint spherical_motor_holder_hip_z_left: origin xyz=-2.7755575615628913511e-17 6.9388939039072283776e-18 -0.051749999999999823919 rpy=1.5707963267948961139 -0.14866879169792920901 1.5707963267948972241 -> xyz=-1.3877787807814456755e-17 -4.0766001685454966719e-17 -0.051749999999999803102 rpy=1.570796326794896558 3.3062838714650006639e-31 1.570796326794896558; type revolute -> fixed
- joint spherical_motor_knee_holder: child cylinder_17 -> cylinder_4; origin xyz=-0.013750000000000095479 0.0024999999999999744649 -0.072000000000000008438 rpy=1.5707963267949001107 -1.5324451476251321758 1.5707963267948763519 -> xyz=-0.013749999999999902925 0.0024999999999999189537 -0.072000000000000008438 rpy=-1.57079632679489678 0.16801524350305055422 -1.5707963267948987784
- joint spherical_shin_left: origin xyz=0.038967453687049846689 -0.092095263467496746301 0 rpy=-1.570796326794896558 0.06472315835280127716 1.5707963267948987784 -> xyz=0.038967453687049791178 -0.092095263467496746301 1.0408340855860842566e-17 rpy=-1.57079632679489678 0.12605142297368143733 1.5707963267949021091
- joint spherical_shin_rod1: origin xyz=0.038967453687039077526 -0.092095263467496801812 1.4988010832439613296e-15 rpy=-1.57079632679489678 -1.3380503778517249813 1.5707963267948987784 -> xyz=0.038967453687049680155 -0.092095263467496857324 5.5511151231257827021e-17 rpy=-1.5707963267948155117 -1.5598420217049260295 1.570796326794971387
- joint uneveral_foot1: origin xyz=0.21747050071614940081 -0.33571800862966422185 0 rpy=-1.5707963267948958919 -1.4835298641951701892 1.5707963267949331954 -> xyz=0.21747050071614937305 -0.33571800862966411083 5.5511151231257827021e-17 rpy=-2.3565428046247982457e-17 -1.5707963267948956698 0
- joint upper_knee: origin xyz=-1.8388068845354155201e-16 0.046751999999999988011 -0.071500000000000563105 rpy=-3.1415926535897855665 -5.3852215752707797424e-15 0.71190954330129141425 -> xyz=1.0755285551056203985e-16 0.046752000000000043523 -0.071499999999999952482 rpy=-3.1415926535897855665 -5.1892128780094199858e-15 0.68585109791284715186
- joint upper_knee_left: origin xyz=-1.3240103458045382467e-13 -0.046752000000042814865 -0.071500000000001479039 rpy=-1.8585155569146270327e-15 2.2316868311075721103e-15 -0.6833117733140818828 -> xyz=5.2041704279304212832e-17 -0.046751999999999988011 -0.071500000000000021871 rpy=-2.905786084916034922e-17 7.0204972010033109187e-17 -0.76652707834254851793
